Commit message: Implemented ros2_control and consistent scripts

File: workspace/src/tractor_description/urdf/tractor.urdf.xacro (robot description, xacro)
@@ -1,269 +1,15 @@
 <?xml version="1.0"?>
 <robot name="mini_tractor" xmlns:xacro="http://www.ros.org/wiki/xacro">
-  <!-- =========================
-       PROPIEDADES GENERALES
-       ========================= -->
-  <xacro:property name="base_length" value="1.00"/>
-  <xacro:property name="base_width"  value="0.70"/>
-  <xacro:property name="base_height" value="0.25"/>
-  <xacro:property name="wheel_radius" value="0.18"/>
-  <xacro:property name="wheel_width"  value="0.08"/>
-  <xacro:property name="camera_size" value="0.08"/>
-  <xacro:property name="wheel_x_front" value="0.30"/>
-  <xacro:property name="wheel_x_rear"  value="-0.30"/>
-  <xacro:property name="wheel_y"       value="0.36"/>
-  <xacro:property name="wheel_z"       value="-0.05"/>
-  <xacro:property name="lidar_radius" value="0.05"/>
-  <xacro:property name="lidar_height" value="0.05"/>
-  <!-- =========================
-       MATERIALES
-       ========================= -->
-  <material name="green">
-    <color rgba="0.1 0.6 0.1 1.0"/>
-  </material>
-  <material name="black">
-    <color rgba="0.1 0.1 0.1 1.0"/>
-  </material>
-  <material name="blue">
-    <color rgba="0.1 0.2 0.8 1.0"/>
-  </material>
-  <!-- =========================
-       LINK RAÍZ DUMMY
-       Evita warning de KDL con inercia en base_link
-       ========================= -->
-  <link name="base_footprint"/>
-  <joint name="base_footprint_joint" type="fixed">
-    <parent link="base_footprint"/>
-    <child link="base_link"/>
-    <origin xyz="0 0 0.18" rpy="0 0 0"/>
-  </joint>
-  <!-- =========================
-       BASE DEL TRACTOR
-       ========================= -->
-  <link name="base_link">
-    <visual>
-      <origin xyz="0 0 0" rpy="0 0 0"/>
-      <geometry>
-        <box size="${base_length} ${base_width} ${base_height}"/>
-      </geometry>
-      <material name="green"/>
-    </visual>
-    <collision>
-      <origin xyz="0 0 0" rpy="0 0 0"/>
-      <geometry>
-        <box size="${base_length} ${base_width} ${base_height}"/>
-      </geometry>
-    </collision>
-    <inertial>
-      <origin xyz="0 0 0" rpy="0 0 0"/>
-      <mass value="40.0"/>
-      <inertia
-        ixx="3.0" ixy="0.0" ixz="0.0"
-        iyy="3.0" iyz="0.0"
-        izz="3.0"/>
-    </inertial>
-  </link>
-  <!-- =========================
-       MACRO DE RUEDA
-       ========================= -->
-  <xacro:macro name="tractor_wheel" params="name x y">
-    <link name="${name}">
-      <visual>
-        <origin xyz="0 0 0" rpy="1.5708 0 0"/>
-        <geometry>
-          <cylinder radius="${wheel_radius}" length="${wheel_width}"/>
-        </geometry>
-        <material name="black"/>
-      </visual>
-      <collision>
-        <origin xyz="0 0 0" rpy="1.5708 0 0"/>
-        <geometry>
-          <cylinder radius="${wheel_radius}" length="${wheel_width}"/>
-        </geometry>
-      </collision>
-      <inertial>
-        <origin xyz="0 0 0" rpy="0 0 0"/>
-        <mass value="2.0"/>
-        <inertia
-          ixx="0.02" ixy="0.0" ixz="0.0"
-          iyy="0.02" iyz="0.0"
-          izz="0.02"/>
-      </inertial>
-    </link>
-    <joint name="${name}_joint" type="continuous">
-      <parent link="base_link"/>
-      <child link="${name}"/>
-      <origin xyz="${x} ${y} ${wheel_z}" rpy="0 0 0"/>
-      <axis xyz="0 1 0"/>
-    </joint>
-  </xacro:macro>
-  <!-- RUEDAS -->
-  <xacro:tractor_wheel name="front_left_wheel"  x="${wheel_x_front}" y="${ wheel_y}"/>
-  <xacro:tractor_wheel name="front_right_wheel" x="${wheel_x_front}" y="${-wheel_y}"/>
-  <xacro:tractor_wheel name="rear_left_wheel"   x="${wheel_x_rear}"  y="${ wheel_y}"/>
-  <xacro:tractor_wheel name="rear_right_wheel"  x="${wheel_x_rear}"  y="${-wheel_y}"/>
-  <!-- =========================
-       CÁMARA
-       ========================= -->
-  <link name="camera_link">
-    <visual>
-      <geometry>
-        <box size="${camera_size} ${camera_size} ${camera_size}"/>
-      </geometry>
-      <material name="blue"/>
-    </visual>
-    <collision>
-      <geometry>
-        <box size="${camera_size} ${camera_size} ${camera_size}"/>
-      </geometry>
-    </collision>
-    <inertial>
-      <mass value="0.5"/>
-      <inertia
-        ixx="0.001" ixy="0.0" ixz="0.0"
-        iyy="0.001" iyz="0.0"
-        izz="0.001"/>
-    </inertial>
-  </link>
-  <joint name="camera_joint" type="fixed">
-    <parent link="base_link"/>
-    <child link="camera_link"/>
-    <origin xyz="0.42 0 0.20" rpy="0 0 0"/>
-  </joint>
-  <!-- =========================
-       LiDAR
-       ========================= -->
-  <link name="lidar_link">
-    <visual>
-      <geometry>
-        <cylinder radius="${lidar_radius}" length="${lidar_height}"/>
-      </geometry>
-      <material name="blue"/>
-    </visual>
-    <collision>
-      <geometry>
-        <cylinder radius="${lidar_radius}" length="${lidar_height}"/>
-      </geometry>
-    </collision>
-    <inertial>
-      <mass value="0.3"/>
-      <inertia
-        ixx="0.001" ixy="0.0" ixz="0.0"
-        iyy="0.001" iyz="0.0"
-        izz="0.001"/>
-    </inertial>
-  </link>
-  <joint name="lidar_joint" type="fixed">
-    <parent link="base_link"/>
-    <child link="lidar_link"/>
-    <origin xyz="0.35 0 0.20" rpy="0 0 0"/>
-  </joint>
-  <!-- =========================
-       GAZEBO: APARIENCIA DE LAS RUEDAS
-       ========================= -->
-  <gazebo reference="base_link">
-    <material>Gazebo/Green</material>
-  </gazebo>
-  <gazebo reference="front_left_wheel">
-    <material>Gazebo/Black</material>
-  </gazebo>
-  <gazebo reference="front_right_wheel">
-    <material>Gazebo/Black</material>
-  </gazebo>
-  <gazebo reference="rear_left_wheel">
-    <material>Gazebo/Black</material>
-  </gazebo>
-  <gazebo reference="rear_right_wheel">
-    <material>Gazebo/Black</material>
-  </gazebo>
-  <!-- =========================
-        DIFF DRIVE SOLO EN RUEDAS TRASERAS
-        ========================= -->
-  <gazebo>
-    <plugin name="tractor_diff_drive" filename="libgazebo_ros_diff_drive.so">
-      <ros>
-        <namespace>/</namespace>
-      </ros>
-      <update_rate>50</update_rate>
-      <left_joint>rear_left_wheel_joint</left_joint>
-      <right_joint>rear_right_wheel_joint</right_joint>
-      <wheel_separation>0.72</wheel_separation>
-      <wheel_diameter>0.36</wheel_diameter>
-      <max_wheel_torque>5.0</max_wheel_torque>
-      <max_wheel_acceleration>1.5</max_wheel_acceleration>
-      <command_topic>cmd_vel</command_topic>
-      <odometry_topic>odom</odometry_topic>
-      <odometry_frame>odom</odometry_frame>
-      <robot_base_frame>base_footprint</robot_base_frame>
-      <publish_odom>true</publish_odom>
-      <publish_odom_tf>true</publish_odom_tf>
-      <publish_wheel_tf>true</publish_wheel_tf>
-    </plugin>
-  </gazebo>
-  <!-- =========================
-       CÁMARA EN GAZEBO
-       ========================= -->
-  <gazebo reference="camera_link">
-    <sensor name="front_camera" type="camera">
-      <always_on>true</always_on>
-      <update_rate>30.0</update_rate>
-      <visualize>true</visualize>
-      <camera>
-        <horizontal_fov>1.3962634</horizontal_fov>
-        <image>
-          <width>640</width>
-          <height>480</height>
-          <format>R8G8B8</format>
-        </image>
-        <clip>
-          <near>0.05</near>
-          <far>50.0</far>
-        </clip>
-      </camera>
-      <plugin name="camera_controller" filename="libgazebo_ros_camera.so">
-        <frame_name>camera_link</frame_name>
-        <camera_name>front_camera</camera_name>
-        <image_topic_name>image_raw</image_topic_name>
-        <camera_info_topic_name>camera_info</camera_info_topic_name>
-      </plugin>
-    </sensor>
-  </gazebo>
-  <!-- =========================
-       LiDAR en Gazebo
-       ========================= -->
-  <gazebo reference="lidar_link">
-    <sensor name="front_lidar" type="ray">
-      <always_on>true</always_on>
-      <update_rate>10.0</update_rate>
-      <visualize>true</visualize>
-      <ray>
-        <scan>
-          <horizontal>
-            <samples>360</samples>
-            <resolution>1</resolution>
-            <min_angle>-1.5708</min_angle>
-            <max_angle>1.5708</max_angle>
-          </horizontal>
-        </scan>
-        <range>
-          <min>0.12</min>
-          <max>8.0</max>
-          <resolution>0.01</resolution>
-        </range>
-        <noise>
-          <type>gaussian</type>
-          <mean>0.0</mean>
-          <stddev>0.01</stddev>
-        </noise>
-      </ray>
-      <plugin name="laser_controller" filename="libgazebo_ros_ray_sensor.so">
-        <ros>
-          <namespace>/</namespace>
-          <remapping>~/out:=/scan</remapping>
-        </ros>
-        <output_type>sensor_msgs/LaserScan</output_type>
-        <frame_name>lidar_link</frame_name>
-      </plugin>
-    </sensor>
-  </gazebo>
+  <xacro:arg
+    name="controllers_file"
+    default="$(find tractor_description)/config/ros2_controllers.yaml"/>
+  <xacro:include filename="$(find tractor_description)/urdf/tractor_properties.xacro"/>
+  <xacro:include filename="$(find tractor_description)/urdf/tractor_core.xacro"/>
+  <xacro:include filename="$(find tractor_description)/urdf/tractor_sensors.xacro"/>
+  <xacro:include filename="$(find tractor_description)/urdf/tractor_ros2_control.xacro"/>
+  <xacro:include filename="$(find tractor_description)/urdf/tractor_gazebo.xacro"/>
+  <xacro:tractor_core/>
+  <xacro:tractor_sensors/>
+  <xacro:tractor_ros2_control/>
+  <xacro:tractor_gazebo controllers_file="$(arg controllers_file)"/>
 </robot>
